Commit message: Add observe named pose and default executor to observe

File: src/sagittarius_arm_ros/sagittarius_moveit/config/sgr532.srdf.xacro (robot description, xacro)
@@ -45,4 +45,12 @@
         <joint name="joint6" value="0"/>
     </group_state>
+    <group_state name="observe" group="sagittarius_arm">
+        <joint name="joint1" value="0.0"/>
+        <joint name="joint2" value="-0.80"/>
+        <joint name="joint3" value="0.85"/>
+        <joint name="joint4" value="0.0"/>
+        <joint name="joint5" value="1.20"/>
+        <joint name="joint6" value="0.0"/>
+    </group_state>
     <group_state name="open" group="sagittarius_gripper">
         <joint name="joint_gripper_left" value="0"/>
